File: design/kicad/soundpad.kicad_sch (KiCad schematic)
At the start: 10 parts, among them J2 Conn_02x18_Counter_Clockwise, K1 Conn_01x01, K2 Conn_01x01, K3 Conn_01x01, K4 Conn_01x01, K5 Conn_01x01, K6 Conn_01x01, K7 Conn_01x01, K8 Conn_01x01, K9 Conn_01x01

Commit message: Adds plate connections to pcb board
Parts:
- J2: symbol Connector_Generic:Conn_02x18_Counter_Clockwise -> Connector_Generic:Conn_02x18_Odd_Even
Connections:
- net at K6.1 (Pin_1): now also J2.11 (Pin_11); no longer J2.6 (Pin_6)
- net at K9.1 (Pin_1): now also J2.17 (Pin_17); no longer J2.9 (Pin_9)
- net at K4.1 (Pin_1): now also J2.7 (Pin_7); no longer J2.4 (Pin_4)
- net at J2.13 (Pin_13): now also K7.1 (Pin_1)
- net at J2.15 (Pin_15): now also K8.1 (Pin_1)
- net at J2.2 (Pin_2): no longer K2.1 (Pin_1)
- net at J2.3 (Pin_3): now also K2.1 (Pin_1); no longer K3.1 (Pin_1)
- net at J2.5 (Pin_5): now also K3.1 (Pin_1); no longer K5.1 (Pin_1)
- net at J2.8 (Pin_8): no longer K8.1 (Pin_1)
- new net: J2.9 (Pin_9), K5.1 (Pin_1)
Changed lines of the file:
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@@
 	)
 	(symbol
-		(lib_id "Connector_Generic:Conn_02x18_Counter_Clockwise")
+		(lib_id "Connector_Generic:Conn_02x18_Odd_Even")
 		(at 153.67 160.02 0)
 		(unit 1)
@@
 			)
 		)
-		(property "Description" "Generic connector, double row, 02x18, counter clockwise pin numbering scheme (similar to DIP package numbering), script generated (kicad-library-utils/schlib/autogen/connector/)"
+		(property "Description" "Generic connector, double row, 02x18, odd/even pin numbering scheme (row 1 odd numbers, row 2 even numbers), script generated (kicad-library-utils/schlib/autogen/connector/)"
 			(at 153.67 160.02 0)
 			(effects
