File: design/kicad/soundpad.kicad_pcb (KiCad board)
At the start: 2 copper layers, 155 x 175 mm, 9 parts, among them J2 Conn_02x18_Counter_Clockwise, K1 Conn_01x01, K2 Conn_01x01, K3 Conn_01x01, K4 Conn_01x01, K5 Conn_01x01, K6 Conn_01x01, K7 Conn_01x01, K8 Conn_01x01

Commit message: completes kicad schematic, starts pcb layout
Parts:
- removed K1, K2, K3, K4, K5, K6, K7, K8: Conn_01x01, TestPoint:TestPoint_Pad_2.5x2.5mm
- added A1: Electrosmith_Daisy_Seed_Rev4, Module:Electrosmith_Daisy_Seed, F.Cu at (112.7, 177.8)
- added C1: 0.1uF, Capacitor_SMD:C_0402_1005Metric, B.Cu at (108.7, 34.0)
- added C10: 0.1uF, Capacitor_SMD:C_0402_1005Metric, F.Cu at (141.4, 138.0)
- added C11: 0.1uF, Capacitor_SMD:C_0402_1005Metric, F.Cu at (100.7, 137.5)
- added C12: 0.1uF, Capacitor_SMD:C_0402_1005Metric, B.Cu at (132.8, 35.9)
- added C13: 10uF, Capacitor_SMD:C_0603_1608Metric, B.Cu at (137.0, 33.8)
- added C14: 0.1uF, Capacitor_SMD:C_0402_1005Metric, F.Cu at (68.4, 146.2)
- added C15: 0.1uF, Capacitor_SMD:C_0402_1005Metric, F.Cu at (262.4, 80.5)
- added C16: 0.1uF, Capacitor_SMD:C_0402_1005Metric, F.Cu at (262.4, 83.0)
- added C17: .47uF, Capacitor_SMD:C_0603_1608Metric, B.Cu at (59.6, 178.4)
- added C18: 0.1uF, Capacitor_SMD:C_0402_1005Metric, B.Cu at (70.2, 182.7)
- added C19: .47uF, Capacitor_SMD:C_0603_1608Metric, B.Cu at (60.8, 175.7)
- added C2: 10uF, Capacitor_SMD:C_0603_1608Metric, B.Cu at (141.6, 31.6)
- added C20: 220UF PANASONIC D8, Capacitor_THT:CP_Radial_D5.0mm_P2.00mm, F.Cu at (75.5, 181.8)
- added C21: 220UF PANASONIC D8, Capacitor_THT:CP_Radial_D5.0mm_P2.00mm, F.Cu at (61.5, 182.0)
- added C23: 0.1uF, Capacitor_SMD:C_0402_1005Metric, B.Cu at (64.6, 178.4)
- added C3: 0.1uF, Capacitor_SMD:C_0402_1005Metric, B.Cu at (117.0, 183.6)
- added C4: 0.1uF, Capacitor_SMD:C_0402_1005Metric, B.Cu at (260.7, 153.2)
- added C5: 0.1uF, Capacitor_SMD:C_0402_1005Metric, B.Cu at (63.2, 138.8)
- added C6: 0.1uF, Capacitor_SMD:C_0402_1005Metric, B.Cu at (105.7, 170.4)
- added C7: 0.1uF, Capacitor_SMD:C_0402_1005Metric, B.Cu at (260.7, 160.7)
- added C8: 0.1uF, Capacitor_SMD:C_0402_1005Metric, B.Cu at (105.0, 51.9)
- added C9: 0.1uF, Capacitor_SMD:C_0402_1005Metric, B.Cu at (260.7, 165.7)
- added D1: 1N4148WS, Diode_SMD:D_SOD-323, B.Cu at (149.0, 192.4)
- added J1: Midi_In, footprints:CUI_SJ1-3553NG, F.Cu at (139.0, 194.5)
- added J10: Clock_Out, footprints:CUI_SJ1-3553NG, F.Cu at (111.0, 194.5)
- added J11: Line_In, footprints:CUI_SJ1-3553NG, F.Cu at (83.0, 194.5)
- added J12: Line_Out, footprints:CUI_SJ1-3553NG, F.Cu at (97.0, 194.4)
- added J15: Conn_01x12_Socket, Connector_PinSocket_1.27mm:PinSocket_1x12_P1.27mm_Vertical, F.Cu at (98.1, 36.5)
- added J16: Conn_01x12_Pin, Connector_PinHeader_1.27mm:PinHeader_1x12_P1.27mm_Vertical_SMD_Pin1Left, F.Cu at (477.3, 144.9)
- added J3: Midi_Out, footprints:CUI_SJ1-3553NG, F.Cu at (125.0, 194.5)
- added J4: Headphone_Out, footprints:CUI_SJ1-3553NG, F.Cu at (69.0, 194.4)
- added J5: Conn_01x12_Socket, Connector_PinSocket_1.27mm:PinSocket_1x12_P1.27mm_Vertical, F.Cu at (161.2, 145.9)
- added J5: Conn_01x12_Socket, Connector_PinSocket_1.27mm:PinSocket_1x12_P1.27mm_Vertical, F.Cu at (277.6, 192.4)
- added J6: Conn_01x12_Socket, Connector_PinSocket_1.27mm:PinSocket_1x12_P1.27mm_Vertical, F.Cu at (93.2, 183.8)
- added J7: Conn_01x12_Socket, Connector_PinSocket_1.27mm:PinSocket_1x12_P1.27mm_Vertical, F.Cu at (46.9, 135.2)
- added J8: Conn_01x09_Pin, Connector_PinHeader_1.27mm:PinHeader_1x09_P1.27mm_Vertical_SMD_Pin1Left, F.Cu at (500.6, 144.8)
- added J9: Conn_01x09_Pin, Connector_PinHeader_1.27mm:PinHeader_1x09_P1.27mm_Vertical_SMD_Pin1Left, F.Cu at (508.6, 144.8)
- added LED_1: White, LED_SMD:LED_PLCC-2_3.4x3.0mm_AK, F.Cu at (55.0, 125.0)
- added LED_10: White, LED_SMD:LED_PLCC-2_3.4x3.0mm_AK, F.Cu at (69.0, 158.1)
- added LED_11: White, LED_SMD:LED_PLCC-2_3.4x3.0mm_AK, F.Cu at (83.0, 158.1)
- added LED_12: White, LED_SMD:LED_PLCC-2_3.4x3.0mm_AK, F.Cu at (97.0, 158.1)
- added LED_13: White, LED_SMD:LED_PLCC-2_3.4x3.0mm_AK, F.Cu at (111.0, 158.1)
- added LED_14: White, LED_SMD:LED_PLCC-2_3.4x3.0mm_AK, F.Cu at (125.0, 158.1)
- added LED_15: White, LED_SMD:LED_PLCC-2_3.4x3.0mm_AK, F.Cu at (139.0, 158.1)
- added LED_16: White, LED_SMD:LED_PLCC-2_3.4x3.0mm_AK, F.Cu at (153.0, 158.1)
- added LED_17: White, LED_SMD:LED_PLCC-2_3.4x3.0mm_AK, F.Cu at (167.9, 173.9)
- added LED_18: White, LED_SMD:LED_PLCC-2_3.4x3.0mm_AK, F.Cu at (168.0, 151.1)
- added LED_19: White, LED_SMD:LED_PLCC-2_3.4x3.0mm_AK, F.Cu at (168.0, 128.3)
- added LED_2: White, LED_SMD:LED_PLCC-2_3.4x3.0mm_AK, F.Cu at (69.0, 125.0)
- added LED_20: White, LED_SMD:LED_PLCC-2_3.4x3.0mm_AK, F.Cu at (40.0, 114.4)
- added LED_21: White, LED_SMD:LED_PLCC-2_3.4x3.0mm_AK, F.Cu at (55.0, 114.5)
- added LED_22: White, LED_SMD:LED_PLCC-2_3.4x3.0mm_AK, F.Cu at (69.0, 114.4)
- added LED_23: White, LED_SMD:LED_PLCC-2_3.4x3.0mm_AK, F.Cu at (83.0, 114.4)
- added LED_24: White, LED_SMD:LED_PLCC-2_3.4x3.0mm_AK, F.Cu at (97.0, 114.4)
- added LED_25: White, LED_SMD:LED_PLCC-2_3.4x3.0mm_AK, F.Cu at (111.0, 114.4)
- added LED_26: White, LED_SMD:LED_PLCC-2_3.4x3.0mm_AK, F.Cu at (125.1, 114.5)
- added LED_27: White, LED_SMD:LED_PLCC-2_3.4x3.0mm_AK, F.Cu at (139.0, 114.5)
- added LED_28: White, LED_SMD:LED_PLCC-2_3.4x3.0mm_AK, F.Cu at (153.0, 114.4)
- added LED_29: White, LED_SMD:LED_PLCC-2_3.4x3.0mm_AK, F.Cu at (168.0, 114.5)
- added LED_3: White, LED_SMD:LED_PLCC-2_3.4x3.0mm_AK, F.Cu at (83.0, 125.1)
- added LED_30: White, LED_SMD:LED_PLCC-2_3.4x3.0mm_AK, F.Cu at (40.0, 57.4)
- added LED_31: White, LED_SMD:LED_PLCC-2_3.4x3.0mm_AK, F.Cu at (40.0, 71.4)
- added LED_32: White, LED_SMD:LED_PLCC-2_3.4x3.0mm_AK, F.Cu at (40.0, 85.5)
- added LED_33: White, LED_SMD:LED_PLCC-2_3.4x3.0mm_AK, F.Cu at (40.0, 99.4)
- added LED_34: White, LED_SMD:LED_PLCC-2_3.4x3.0mm_AK, F.Cu at (168.0, 57.4)
- added LED_35: White, LED_SMD:LED_PLCC-2_3.4x3.0mm_AK, F.Cu at (168.0, 71.4)
- added LED_36: White, LED_SMD:LED_PLCC-2_3.4x3.0mm_AK, F.Cu at (168.0, 85.4)
- added LED_37: White, LED_SMD:LED_PLCC-2_3.4x3.0mm_AK, F.Cu at (168.0, 99.4)
- added LED_38: White, LED_SMD:LED_PLCC-2_3.4x3.0mm_AK, F.Cu at (57.0, 43.5)
- added LED_39: White, LED_SMD:LED_PLCC-2_3.4x3.0mm_AK, F.Cu at (71.0, 43.5)
- added LED_4: White, LED_SMD:LED_PLCC-2_3.4x3.0mm_AK, F.Cu at (97.0, 125.1)
- added LED_40: White, LED_SMD:LED_PLCC-2_3.4x3.0mm_AK, F.Cu at (85.0, 43.5)
- added LED_41: White, LED_SMD:LED_PLCC-2_3.4x3.0mm_AK, F.Cu at (99.0, 43.5)
- added LED_42: White, LED_SMD:LED_PLCC-2_3.4x3.0mm_AK, F.Cu at (113.0, 43.8)
- added LED_43: White, LED_SMD:LED_PLCC-2_3.4x3.0mm_AK, F.Cu at (-102.7, 57.6)
- added LED_44: White, LED_SMD:LED_PLCC-2_3.4x3.0mm_AK, F.Cu at (-102.7, 62.3)
- added LED_45: White, LED_SMD:LED_PLCC-2_3.4x3.0mm_AK, F.Cu at (-102.7, 67.1)
- added LED_46: White, LED_SMD:LED_PLCC-2_3.4x3.0mm_AK, F.Cu at (-102.7, 71.8)
- added LED_47: White, LED_SMD:LED_PLCC-2_3.4x3.0mm_AK, F.Cu at (-102.7, 76.6)
- added LED_48: White, LED_SMD:LED_PLCC-2_3.4x3.0mm_AK, F.Cu at (-102.7, 81.3)
- added LED_5: White, LED_SMD:LED_PLCC-2_3.4x3.0mm_AK, F.Cu at (111.0, 125.1)
- added LED_6: White, LED_SMD:LED_PLCC-2_3.4x3.0mm_AK, F.Cu at (125.0, 125.1)
- added LED_7: White, LED_SMD:LED_PLCC-2_3.4x3.0mm_AK, F.Cu at (139.0, 125.1)
- added LED_8: White, LED_SMD:LED_PLCC-2_3.4x3.0mm_AK, F.Cu at (153.0, 125.1)
- added LED_9: White, LED_SMD:LED_PLCC-2_3.4x3.0mm_AK, F.Cu at (55.0, 158.1)
- added MK1: Microphone, soundpad_library:AOM-5024L-HD-R, F.Cu at (539.6, 146.0)
- added MK2: Microphone, soundpad_library:AOM-5024L-HD-R, F.Cu at (554.4, 169.8)
- added MicL1: Conn_01x01, TestPoint:TestPoint_Pad_2.5x2.5mm, F.Cu at (490.8, 153.9)
- added MicR1: Conn_01x01, TestPoint:TestPoint_Pad_2.5x2.5mm, F.Cu at (490.8, 158.4)
- added Pad1: Conn_01x01, TestPoint:TestPoint_Pad_2.5x2.5mm, F.Cu at (490.8, 163.0)
- added Pad10: Conn_01x01, TestPoint:TestPoint_Pad_2.5x2.5mm, F.Cu at (495.4, 176.7)
- added Pad11: Conn_01x01, TestPoint:TestPoint_Pad_2.5x2.5mm, F.Cu at (499.9, 153.9)
- added Pad12: Conn_01x01, TestPoint:TestPoint_Pad_2.5x2.5mm, F.Cu at (499.9, 158.4)
- added Pad13: Conn_01x01, TestPoint:TestPoint_Pad_2.5x2.5mm, F.Cu at (499.9, 163.0)
- added Pad14: Conn_01x01, TestPoint:TestPoint_Pad_2.5x2.5mm, F.Cu at (499.9, 167.6)
- added Pad15: Conn_01x01, TestPoint:TestPoint_Pad_2.5x2.5mm, F.Cu at (499.9, 172.1)
- added Pad16: Conn_01x01, TestPoint:TestPoint_Pad_2.5x2.5mm, F.Cu at (499.9, 176.7)
- added Pad19: Conn_01x01, TestPoint:TestPoint_Pad_2.5x2.5mm, F.Cu at (504.4, 153.9)
- added Pad2: Conn_01x01, TestPoint:TestPoint_Pad_2.5x2.5mm, F.Cu at (490.8, 167.6)
- added Pad3: Conn_01x01, TestPoint:TestPoint_Pad_2.5x2.5mm, F.Cu at (490.8, 172.1)
- added Pad4: Conn_01x01, TestPoint:TestPoint_Pad_2.5x2.5mm, F.Cu at (490.8, 176.7)
- added Pad5: Conn_01x01, TestPoint:TestPoint_Pad_2.5x2.5mm, F.Cu at (495.4, 153.9)
- added Pad6: Conn_01x01, TestPoint:TestPoint_Pad_2.5x2.5mm, F.Cu at (495.4, 158.4)
- added Pad7: Conn_01x01, TestPoint:TestPoint_Pad_2.5x2.5mm, F.Cu at (495.4, 163.0)
- added Pad8: Conn_01x01, TestPoint:TestPoint_Pad_2.5x2.5mm, F.Cu at (495.4, 167.6)
- added Pad9: Conn_01x01, TestPoint:TestPoint_Pad_2.5x2.5mm, F.Cu at (495.4, 172.1)
- added PadAfter1: Conn_01x01, TestPoint:TestPoint_Pad_2.5x2.5mm, F.Cu at (504.4, 158.4)
- added PadEmpty1: Conn_01x01, TestPoint:TestPoint_Pad_2.5x2.5mm, F.Cu at (504.4, 163.0)
- added PadFlow1: Conn_01x01, TestPoint:TestPoint_Pad_2.5x2.5mm, F.Cu at (504.4, 167.6)
- added PadGroups1: Conn_01x01, TestPoint:TestPoint_Pad_2.5x2.5mm, F.Cu at (504.4, 172.1)
- added PadL1: Conn_01x01, TestPoint:TestPoint_Pad_2.5x2.5mm, F.Cu at (504.4, 176.7)
- added PadL2: Conn_01x01, TestPoint:TestPoint_Pad_2.5x2.5mm, F.Cu at (509.0, 153.9)
- added PadL3: Conn_01x01, TestPoint:TestPoint_Pad_2.5x2.5mm, F.Cu at (509.0, 158.4)
- added PadL4: Conn_01x01, TestPoint:TestPoint_Pad_2.5x2.5mm, F.Cu at (509.0, 163.0)
- added PadMod1: Conn_01x01, TestPoint:TestPoint_Pad_2.5x2.5mm, F.Cu at (509.0, 167.6)
- added PadNotes1: Conn_01x01, TestPoint:TestPoint_Pad_2.5x2.5mm, F.Cu at (509.0, 172.1)
- added PadPocket1: Conn_01x01, TestPoint:TestPoint_Pad_2.5x2.5mm, F.Cu at (509.0, 176.7)
- added PadR1: Conn_01x01, TestPoint:TestPoint_Pad_2.5x2.5mm, F.Cu at (513.5, 153.9)
- added PadR2: Conn_01x01, TestPoint:TestPoint_Pad_2.5x2.5mm, F.Cu at (513.5, 158.4)
- added PadR3: Conn_01x01, TestPoint:TestPoint_Pad_2.5x2.5mm, F.Cu at (513.5, 163.0)
- added PadR4: Conn_01x01, TestPoint:TestPoint_Pad_2.5x2.5mm, F.Cu at (513.5, 167.6)
- added PadSet1: Conn_01x01, TestPoint:TestPoint_Pad_2.5x2.5mm, F.Cu at (513.5, 172.1)
- added PadVelo1: Conn_01x01, TestPoint:TestPoint_Pad_2.5x2.5mm, F.Cu at (513.5, 176.7)
- added R1: 10K, Resistor_SMD:R_0603_1608Metric, B.Cu at (156.2, 46.8)
- added R10: 4.7K, Resistor_SMD:R_0603_1608Metric, F.Cu at (152.3, 136.5)
- added R11: 75k, Resistor_SMD:R_0603_1608Metric, B.Cu at (61.7, 140.8)
- added R12: 100k, Resistor_SMD:R_0603_1608Metric, B.Cu at (65.1, 137.4)
- added R13: 10k, Resistor_SMD:R_0603_1608Metric, B.Cu at (256.7, 155.7)
- added R14: 10k, Resistor_SMD:R_0603_1608Metric, B.Cu at (256.7, 158.2)
- added R15: 10k, Resistor_SMD:R_0603_1608Metric, B.Cu at (256.7, 160.7)
- added R16: 100k, Resistor_SMD:R_0603_1608Metric, B.Cu at (107.0, 170.4)
- added R17: 10k, Resistor_SMD:R_0603_1608Metric, B.Cu at (256.7, 165.7)
- added R18: 75k, Resistor_SMD:R_0603_1608Metric, B.Cu at (108.7, 172.4)
- added R19: 10k, Resistor_SMD:R_0603_1608Metric, B.Cu at (252.7, 153.2)
- added R2: DI*, Resistor_THT:R_Axial_DIN0204_L3.6mm_D1.6mm_P5.08mm_Horizontal, F.Cu at (138.1, 41.8)
- added R20: 100k, Resistor_SMD:R_0603_1608Metric, B.Cu at (103.0, 52.4)
- added R21: 10k, Resistor_SMD:R_0603_1608Metric, B.Cu at (252.7, 158.2)
- added R22: 75k, Resistor_SMD:R_0603_1608Metric, B.Cu at (252.7, 160.7)
- added R23: 140R, Resistor_SMD:R_0603_1608Metric, F.Cu at (101.4, 125.1)
- added R24: 4.7K, Resistor_SMD:R_0603_1608Metric, F.Cu at (151.7, 135.1)
- added R25: 140R, Resistor_SMD:R_0603_1608Metric, F.Cu at (115.0, 125.0)
- added R26: 140R, Resistor_SMD:R_0603_1608Metric, F.Cu at (126.3, 128.7)
- added R27: 140R, Resistor_SMD:R_0603_1608Metric, F.Cu at (143.0, 125.0)
- added R28: 140R, Resistor_SMD:R_0603_1608Metric, F.Cu at (152.6, 127.9)
- added R29: 140R, Resistor_SMD:R_0603_1608Metric, F.Cu at (59.7, 158.0)
- added R3: 220R, Resistor_SMD:R_0603_1608Metric, B.Cu at (147.0, 192.8)
- added R30: 140R, Resistor_SMD:R_0603_1608Metric, F.Cu at (70.5, 154.6)
- added R31: 140R, Resistor_SMD:R_0603_1608Metric, F.Cu at (87.7, 158.0)
- added R32: 140R, Resistor_SMD:R_0603_1608Metric, F.Cu at (98.5, 154.6)
- added R33: 140R, Resistor_SMD:R_0603_1608Metric, F.Cu at (112.4, 154.5)
- added R34: 140R, Resistor_SMD:R_0603_1608Metric, F.Cu at (129.0, 157.2)
- added R35: 140R, Resistor_SMD:R_0603_1608Metric, F.Cu at (142.6, 157.2)
- added R36: 140R, Resistor_SMD:R_0603_1608Metric, F.Cu at (149.4, 157.3)
- added R37: 4.7K, Resistor_SMD:R_0603_1608Metric, F.Cu at (111.5, 136.1)
- added R38: 4.7K, Resistor_SMD:R_0603_1608Metric, F.Cu at (110.7, 134.5)
- added R39: 140R, Resistor_SMD:R_0603_1608Metric, F.Cu at (164.1, 173.9)
- added R4: 33R, Resistor_SMD:R_0603_1608Metric, F.Cu at (51.0, 150.9)
- added R40: 140R, Resistor_SMD:R_0603_1608Metric, F.Cu at (163.8, 151.2)
- added R41: 140R, Resistor_SMD:R_0603_1608Metric, F.Cu at (163.6, 128.2)
- added R42: 140R, Resistor_SMD:R_0603_1608Metric, F.Cu at (41.5, 117.8)
- added R43: 140R, Resistor_SMD:R_0603_1608Metric, F.Cu at (59.1, 115.5)
- added R44: 140R, Resistor_SMD:R_0603_1608Metric, F.Cu at (73.6, 115.3)
- added R45: 140R, Resistor_SMD:R_0603_1608Metric, F.Cu at (87.4, 115.2)
- added R46: 140R, Resistor_SMD:R_0603_1608Metric, F.Cu at (101.1, 114.4)
- added R47: 140R, Resistor_SMD:R_0603_1608Metric, F.Cu at (115.1, 115.0)
- added R48: 140R, Resistor_SMD:R_0603_1608Metric, F.Cu at (129.7, 114.5)
- added R49: 140R, Resistor_SMD:R_0603_1608Metric, F.Cu at (143.0, 114.4)
- added R5: 10R, Resistor_SMD:R_0603_1608Metric, B.Cu at (134.5, 184.4)
- added R50: 140R, Resistor_SMD:R_0603_1608Metric, F.Cu at (153.4, 118.0)
- added R51: 140R, Resistor_SMD:R_0603_1608Metric, F.Cu at (164.0, 114.4)
- added R52: 140R, Resistor_SMD:R_0603_1608Metric, F.Cu at (41.5, 60.8)
- added R53: 140R, Resistor_SMD:R_0603_1608Metric, F.Cu at (41.6, 75.0)
- added R54: 140R, Resistor_SMD:R_0603_1608Metric, F.Cu at (41.5, 89.2)
- added R55: 2.2K, Resistor_SMD:R_0603_1608Metric, B.Cu at (129.4, 34.5)
- added R55: 2.2K, Resistor_SMD:R_0603_1608Metric, B.Cu at (131.3, 34.5)
- added R56: 50R, Resistor_SMD:R_0603_1608Metric, B.Cu at (108.3, 31.6)
- added R56: 50R, Resistor_SMD:R_0603_1608Metric, B.Cu at (106.4, 31.6)
- added R57: 47k, Resistor_SMD:R_0603_1608Metric, F.Cu at (232.6, 100.0)
- added R58: 47k, Resistor_SMD:R_0603_1608Metric, F.Cu at (236.2, 102.6)
- added R59: 47k, Resistor_SMD:R_0603_1608Metric, F.Cu at (49.4, 184.4)
- added R6: 270R, Resistor_SMD:R_0603_1608Metric, F.Cu at (227.2, 106.0)
- added R60: 47k, Resistor_SMD:R_0603_1608Metric, F.Cu at (229.2, 90.8)
- added R61: 47k, Resistor_SMD:R_0603_1608Metric, F.Cu at (247.2, 98.2)
- added R62: 100K, Resistor_SMD:R_0603_1608Metric, B.Cu at (147.4, 35.8)
- added R63: 100K, Resistor_SMD:R_0603_1608Metric, B.Cu at (149.8, 33.7)
- added R64: DI*, Resistor_THT:R_Axial_DIN0204_L3.6mm_D1.6mm_P5.08mm_Horizontal, F.Cu at (140.5, 46.8)
- added R65: 2.2K, Resistor_SMD:R_0603_1608Metric, B.Cu at (110.7, 33.2)
- added R66: 50R, Resistor_SMD:R_0603_1608Metric, B.Cu at (135.9, 36.5)
- added R67: 100K, Resistor_SMD:R_0603_1608Metric, B.Cu at (147.6, 39.1)
- added R68: 100K, Resistor_SMD:R_0603_1608Metric, B.Cu at (135.2, 33.8)
- added R69: 10K, Resistor_SMD:R_0603_1608Metric, B.Cu at (157.8, 44.0)
- added R7: 140R, Resistor_SMD:R_0603_1608Metric, F.Cu at (58.9, 125.9)
- added R70: DI*, Resistor_THT:R_Axial_DIN0204_L3.6mm_D1.6mm_P5.08mm_Horizontal, F.Cu at (150.4, 40.5)
- added R71: DI*, Resistor_THT:R_Axial_DIN0204_L3.6mm_D1.6mm_P5.08mm_Horizontal, F.Cu at (153.2, 45.6)
- added R72: 140R, Resistor_SMD:R_0603_1608Metric, F.Cu at (41.5, 103.0)
- added R73: 140R, Resistor_SMD:R_0603_1608Metric, F.Cu at (163.6, 57.4)
- added R74: 140R, Resistor_SMD:R_0603_1608Metric, F.Cu at (163.6, 71.4)
- added R75: 140R, Resistor_SMD:R_0603_1608Metric, F.Cu at (164.0, 85.4)
- added R76: 140R, Resistor_SMD:R_0603_1608Metric, F.Cu at (166.5, 103.0)
- added R77: 140R, Resistor_SMD:R_0603_1608Metric, F.Cu at (61.2, 44.2)
- added R78: 140R, Resistor_SMD:R_0603_1608Metric, F.Cu at (74.8, 43.4)
- added R79: 140R, Resistor_SMD:R_0603_1608Metric, F.Cu at (88.8, 43.5)
- added R8: 140R, Resistor_SMD:R_0603_1608Metric, F.Cu at (72.8, 125.9)
- added R80: 140R, Resistor_SMD:R_0603_1608Metric, F.Cu at (102.8, 43.6)
- added R81: 140R, Resistor_SMD:R_0603_1608Metric, F.Cu at (109.4, 43.8)
- added R82: 140R, Resistor_SMD:R_0603_1608Metric, F.Cu at (-97.6, 56.5)
- added R83: 140R, Resistor_SMD:R_0603_1608Metric, F.Cu at (-97.6, 59.0)
- added R84: 140R, Resistor_SMD:R_0603_1608Metric, F.Cu at (-97.6, 61.5)
- added R85: 140R, Resistor_SMD:R_0603_1608Metric, F.Cu at (-97.6, 64.0)
- added R86: 140R, Resistor_SMD:R_0603_1608Metric, F.Cu at (-97.6, 66.5)
- added R87: 140R, Resistor_SMD:R_0603_1608Metric, F.Cu at (-97.6, 69.0)
- added R88: 4.7K, Resistor_SMD:R_0603_1608Metric, F.Cu at (56.7, 147.3)
- added R89: 4.7K, Resistor_SMD:R_0603_1608Metric, F.Cu at (57.6, 148.9)
- added R9: 140R, Resistor_SMD:R_0603_1608Metric, F.Cu at (84.6, 128.7)
- added R90: 10k, Resistor_SMD:R_0603_1608Metric, F.Cu at (262.4, 85.5)
- added R91: 100k, Resistor_SMD:R_0603_1608Metric, F.Cu at (262.4, 88.0)
- added R92: 10k, Resistor_SMD:R_0603_1608Metric, F.Cu at (262.4, 90.5)
- added R93: 75k, Resistor_SMD:R_0603_1608Metric, F.Cu at (262.4, 93.0)
- added R94: 22K, Resistor_SMD:R_0603_1608Metric, B.Cu at (61.9, 179.8)
- added R95: 33K, Resistor_SMD:R_0603_1608Metric, B.Cu at (64.1, 180.9)
- added R97: 22K, Resistor_SMD:R_0603_1608Metric, B.Cu at (63.5, 173.7)
- added R98: 33K, Resistor_SMD:R_0603_1608Metric, B.Cu at (68.0, 174.9)
- added RV1: slider2, Potentiometer_THT:Potentiometer_Bourns_PTA6043_Single_Slide, F.Cu at (119.5, 73.3)
- added RV2: slider3, Potentiometer_THT:Potentiometer_Bourns_PTA6043_Single_Slide, F.Cu at (119.5, 87.2)
- added RV3: sliderA, Potentiometer_THT:Potentiometer_Bourns_PTA4543_Single_Slide, F.Cu at (124.5, 107.8)
- added RV4: slider1, Potentiometer_THT:Potentiometer_Bourns_PTA6043_Single_Slide, F.Cu at (119.5, 59.2)
- added RV5: slider4, Potentiometer_THT:Potentiometer_Bourns_PTA6043_Single_Slide, F.Cu at (119.5, 101.2)
- added RV6: sliderB, Potentiometer_THT:Potentiometer_Bourns_PTA4543_Single_Slide, F.Cu at (134.6, 107.8)
- added RV7: sliderC, Potentiometer_THT:Potentiometer_Bourns_PTA4543_Single_Slide, F.Cu at (144.6, 107.8)
- added RV9: sliderD, Potentiometer_THT:Potentiometer_Bourns_PTA4543_Single_Slide, F.Cu at (154.7, 107.8)
- added SW1: SW_DPDT_x2, soundpad_library:Toggle Submini DPDT Prongs, F.Cu at (131.0, 42.0)
- added TF1: TF-CARD H1.8, soundpad_library:TF-SMD_TF-CARD-H1.8, B.Cu at (49.8, 190.9)
- added U**1: LM4881MX SOIC-8, Package_SO:SOIC-8_3.9x4.9mm_P1.27mm, B.Cu at (69.1, 179.5)
- added U1: MCP6002-xSN, Package_SO:SOIC-8_3.9x4.9mm_P1.27mm, B.Cu at (141.6, 35.1)
- added U10: MPR121QR2, Package_DFN_QFN:UQFN-20_3x3mm_P0.4mm, B.Cu at (146.1, 140.3)
- added U2: H11L1S(TA), footprints:H11L1STA_EVE, B.Cu at (154.0, 191.0)
- added U3: PCA9685PW, Package_SO:TSSOP-28_4.4x9.7mm_P0.65mm, F.Cu at (146.9, 141.6)
- added U4: MPR121QR2, Package_DFN_QFN:UQFN-20_3x3mm_P0.4mm, B.Cu at (61.4, 136.1)
- added U5: MPR121QR2, Package_DFN_QFN:UQFN-20_3x3mm_P0.4mm, B.Cu at (100.5, 171.3)
- added U6: MPR121QR2, Package_DFN_QFN:UQFN-20_3x3mm_P0.4mm, B.Cu at (103.8, 44.8)
- added U7: PCA9685PW, Package_SO:TSSOP-28_4.4x9.7mm_P0.65mm, F.Cu at (105.6, 141.1)
- added U8: PCA9685PW, Package_SO:TSSOP-28_4.4x9.7mm_P0.65mm, F.Cu at (63.2, 142.6)
- added U9: MCP6002-xSN, Package_SO:SOIC-8_3.9x4.9mm_P1.27mm, B.Cu at (82.6, 182.9)
- added USBC1: TYPE-C-31-M-12, Connector_USB:USB_C_Receptacle_HRO_TYPE-C-31-M-12, F.Cu at (166.9, 195.5)
- added VR1: RK10J12R0A0B, footprints:RK10J12R0A0B, F.Cu at (170.8, 43.6)
- added VR2: RK10J12R0A0B, footprints:RK10J12R0A0B, F.Cu at (37.5, 43.5)
- J2: value Conn_02x18_Counter_Clockwise -> Conn_01x09_Pin; footprint Connector_PinHeader_2.54mm:PinHeader_2x18_P2.54mm_Vertical_SMD -> Connector_PinHeader_1.27mm:PinHeader_1x09_P1.27mm_Vertical_SMD_Pin1Left
- moved J2 422.4 mm to (492.6, 144.8), turned to 0 degrees
Connections:
- J2 pad 2: unconnected-(J2-Pin_2-Pad2) -> Net-(J2-Pin_2)
- J2 pad 4: unconnected-(J2-Pin_4-Pad4) -> Net-(J2-Pin_4)
- J2 pad 6: unconnected-(J2-Pin_6-Pad6) -> Net-(J2-Pin_6)
- J2 pad 8: unconnected-(J2-Pin_8-Pad8) -> Net-(J2-Pin_8)
Routing:
- net Audio_out_1: track 0.00 -> 241.8 mm, vias 0 -> 1
- net /IO_SDcard/Line_In_R: track 0.00 -> 223.5 mm
- net /IO_SDcard/Line_In_L: track 0.00 -> 220.1 mm
- net Audio_out_2: track 0.00 -> 210.6 mm, vias 0 -> 1
- net SDA: track 0.00 -> 190.1 mm, vias 0 -> 3
- net /Audio_IO/Headphone_Wiper_L: track 0.00 -> 179.3 mm, vias 0 -> 1
- net SCL: track 0.00 -> 178.6 mm, vias 0 -> 3
- net /Audio_IO/Headphone_Wiper_R: track 0.00 -> 177.0 mm, vias 0 -> 1
- net 3V3_A: track 0.00 -> 158.0 mm
- net GND: track 0.00 -> 127.3 mm, vias 0 -> 15
- net /LEDs/LED_39: track 0.00 -> 107.5 mm
- net /LEDs/LED_40: track 0.00 -> 103.2 mm
- net /LEDs/LED_41: track 0.00 -> 100.0 mm
- net /LEDs/LED_42: track 0.00 -> 98.2 mm
- net /LEDs/LED_38: track 0.00 -> 96.6 mm
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- added copper zone on In1.Cu, net 5V
Other:
- board size 155 x 175 mm -> 144 x 168 mm
- copper layers 2 -> 4
- board text added: "{dblquote}Knob operating potentiometers{dblquote} smd straight to via because through hole with audio taper not in stock"
- board text removed: "POUCH"

Commit message: routes PCB all except PWR
Parts:
- removed the J5 at (161.2, 145.9)
- removed the J5 at (277.6, 192.4)
- removed LED_43, LED_44, LED_45, LED_46, LED_47, LED_48: White, LED_SMD:LED_PLCC-2_3.4x3.0mm_AK
- removed R13, R14, R15, R17, R19, R21, R90, R92: 10k, Resistor_SMD:R_0603_1608Metric
- removed R82, R83, R84, R85, R86, R87: 140R, Resistor_SMD:R_0603_1608Metric
- added J5: Conn_01x12_Socket, Connector_PinSocket_1.27mm:PinSocket_1x12_P1.27mm_Vertical, F.Cu at (160.4, 145.9)
- added R96: 10k, Resistor_SMD:R_0603_1608Metric, B.Cu at (109.6, 165.3)
- added R99: 10k, Resistor_SMD:R_0603_1608Metric, B.Cu at (107.9, 163.7)
- C15, C16, C20, J12, R4, R57, R58, R59, R6, R60, R61, R91, R93: moved to B.Cu
- C17, C18, C19, C23, C8, C9, R20, R22, R5, R94, R95, R97, R98, U**1, U6, U9: moved to F.Cu
- moved C9 227.2 mm to (72.1, 39.1), turned to 90 degrees
- moved R22 210.0 mm to (82.1, 38.2)
- moved R61 209.1 mm to (55.3, 181.1), turned to 90 degrees
- moved R57 202.3 mm to (47.5, 181.5), turned to 90 degrees
- moved R58 202.2 mm to (48.6, 178.2), turned to 90 degrees
- moved C4 198.7 mm to (63.1, 132.4), turned to -90 degrees
- moved R60 195.6 mm to (54.2, 178.1), turned to 90 degrees
- moved C7 163.3 mm to (97.6, 169.2), turned to -90 degrees
- moved C16 130.0 mm to (142.7, 133.7), turned to 90 degrees
- moved C15 128.8 mm to (142.6, 127.8), turned to 180 degrees
- moved R91 128.0 mm to (140.5, 127.2), turned to -90 degrees
- moved R93 122.9 mm to (143.9, 125.5), turned to -90 degrees
- moved R6 108.3 mm to (151.4, 183.3)
- moved R4 82.0 mm to (122.9, 190.4), turned to 0 degrees
- moved C3 38.2 mm to (155.3, 184.2), turned to 0 degrees
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Connections:
- U10 pad 10: FILT -> PadEmpty
- U10 pad 11: MOD -> POUCH
- U10 pad 12: POUCH -> SCRATCH
- U10 pad 13: SCRATCH -> COMP
- U10 pad 14: COMP -> EFFCT
- U10 pad 15: EFFCT -> Pad5
- U10 pad 16: Extra1 -> Pad6
- U10 pad 17: Extra2 -> Pad7
- U10 pad 18: Extra3 -> Pad8
- U10 pad 19: unconnected-(U10-LED7/ELE11-Pad19) -> PadGroups
- U10 pad 2: Net-(U10-SCL) -> SCL
- U10 pad 8: SOUND -> PadR3
- U10 pad 9: AMP -> PadR4
- U3 pad 12: /LEDs/LED_14 -> unconnected-(U3-LED6-Pad12)
- U3 pad 6: /LEDs/LED_26 -> unconnected-(U3-LED0-Pad6)
- U6 pad 10: PadR3 -> unconnected-(U6-ELE2-Pad10)
- U6 pad 11: PadR4 -> PadFlow
- U6 pad 12: PadAfter -> PadMod
- U6 pad 14: PadMod -> PadAfter
- U6 pad 15: PadSet -> PadL2
- U6 pad 16: PadEmpty -> PadL1
- U6 pad 17: PadFlow -> unconnected-(U6-LED5/ELE9-Pad17)
- U7 pad 10: /LEDs/LED_39 -> unconnected-(U7-LED4-Pad10)
- U7 pad 9: /LEDs/LED_39 -> /LEDs/LED_4
- USBC1 pad A1: unconnected-(USBC1-GND-PadA1) -> GND
Routing:
- net SDA: track 190.1 -> 1006.1 mm, vias 3 -> 0
- net SCL: track 178.6 -> 898.9 mm, vias 3 -> 0
- net GND: track 127.3 -> 377.5 mm, vias 15 -> 28
- net Audio_in_1: track 0.00 -> 237.8 mm
- net SD_CK: track 0.00 -> 167.3 mm
- net Audio_in_2: track 0.00 -> 156.0 mm
- net Net-(A1-ADC_0): track 0.00 -> 131.3 mm
- net Net-(A1-ADC_1): track 0.00 -> 125.0 mm
- net Net-(A1-ADC_2): track 0.00 -> 119.4 mm
- net SD_D1: track 0.00 -> 118.3 mm
- net SD_D0: track 0.00 -> 117.1 mm
- net Net-(A1-ADC_3): track 0.00 -> 113.9 mm
- net SD_CMD: track 0.00 -> 94.5 mm
- net Net-(A1-ADC_4): track 0.00 -> 93.2 mm
- net SD_D2: track 0.00 -> 85.8 mm
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- added copper zone on In2.Cu, net GND

Commit message: PCB all routed, Moves top components to top file
Parts:
- removed J16: Conn_01x12_Pin, Connector_PinHeader_1.27mm:PinHeader_1x12_P1.27mm_Vertical_SMD_Pin1Left
- removed J2, J8, J9: Conn_01x09_Pin, Connector_PinHeader_1.27mm:PinHeader_1x09_P1.27mm_Vertical_SMD_Pin1Left
- removed MK1, MK2: Microphone, soundpad_library:AOM-5024L-HD-R
- removed MicL1, MicR1, Pad1, Pad10, Pad11, Pad12, Pad13, Pad14, Pad15, Pad16, Pad19, Pad2, Pad3, Pad4, Pad5, Pad6, Pad7, Pad8, Pad9, PadAfter1, PadEmpty1, PadFlow1, PadGroups1, PadL1, PadL2, PadL3, PadL4, PadMod1, PadNotes1, PadPocket1, PadR1, PadR2, PadR3, PadR4, PadSet1, PadVelo1: Conn_01x01, TestPoint:TestPoint_Pad_2.5x2.5mm
- moved R65 12.1 mm to (126.0, 34.5)
- moved C1 12.1 mm to (123.4, 34.8)
- moved C16 4.35 mm to (145.1, 137.3)
- moved C11 1.08 mm to (99.6, 137.5)
Connections:
- USBC1 pad A4: unconnected-(USBC1-VBUS-PadA4) -> 5V
- USBC1 pad B6: unconnected-(USBC1-DP2-PadB6) -> D+
- USBC1 pad B7: unconnected-(USBC1-DN2-PadB7) -> D-
- USBC1 pad B9: unconnected-(USBC1-VBUS-PadB9) -> 5V
Routing:
- net 3V3_D: track 18.8 -> 415.4 mm, vias 0 -> 6
- net 3V3_A: track 175.5 -> 340.2 mm, vias 0 -> 1
- net D+: track 65.0 -> 100.4 mm
- net 5V: track 87.9 -> 114.4 mm, vias 48 -> 50
- net Net-(C1-Pad2): track 12.3 -> 32.5 mm
- net MicR: track 54.4 -> 43.6 mm
- net SD_D0: track 117.1 -> 124.3 mm
- net SD_D1: track 118.3 -> 121.8 mm
- net Net-(LED_5-K): track 0.00 -> 2.87 mm
- net Net-(LED_3-K): track 0.00 -> 2.82 mm
- net Net-(LED_25-K): track 0.00 -> 2.72 mm
- net Audio_in_1: track 237.8 -> 235.4 mm
- net unconnected-(VR1-1/1-Pad1): track 1.82 -> 0.00 mm, vias 1 -> 0
- net MicL: track 17.3 -> 15.7 mm
- net /LEDs/LED_25: track 36.0 -> 34.4 mm
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