File: design/kicad/leds.kicad_sch (KiCad schematic)
At the start: 96 parts, among them U3 PCA9685PW, U7 PCA9685PW, U8 PCA9685PW

Commit message: last commit before refactor repo: kicad mostly
Parts:
- removed C10, C11, C14: 0.1uF, Capacitor_SMD:C_0402_1005Metric, symbol Device:C
- removed LED_1, LED_10, LED_11, LED_12, LED_13, LED_14, LED_15, LED_16, LED_17, LED_18, LED_19, LED_2, LED_20, LED_21, LED_22, LED_23, LED_24, LED_25, LED_26, LED_27, LED_28, LED_29, LED_3, LED_30, LED_31, LED_32, LED_33, LED_34, LED_35, LED_36, LED_37, LED_38, LED_39, LED_4, LED_40, LED_41, LED_42, LED_5, LED_6, LED_7, LED_8, LED_9: White, LED_SMD:LED_PLCC-2_3.4x3.0mm_AK, symbol Device:LED
- removed R10, R24, R37, R38, R88, R89: 4.7K, Resistor_SMD:R_0603_1608Metric, symbol Device:R
- removed R23, R25, R26, R27, R28, R29, R30, R31, R32, R33, R34, R35, R36, R39, R40, R41, R42, R43, R44, R45, R46, R47, R48, R49, R50, R51, R52, R53, R54, R72, R73, R74, R75, R76, R77, R78, R79, R80, R81, R9: 150R, Resistor_SMD:R_0603_1608Metric, symbol Device:R
- removed U3, U7, U8: PCA9685PW, Package_SO:TSSOP-28_4.4x9.7mm_P0.65mm, symbol Driver_LED:PCA9685PW
- added C1: 0.1uF, Capacitor_SMD:C_0402_1005Metric, symbol Device:C
- added D2, D4: LED, LED_THT:LED_D5.0mm, symbol Device:LED
- added D5: LED, LED_THT:LED_D3.0mm, symbol Device:LED
- added Eraser1, Play_Paper1, Play_Point1, Play_Pouch1, Rec_Paper1, Rec_Point1, Rec_Pouch1, Smudger1: Cherry-MX-RGB-0603, CherryMX:Cherry-MX-RGB-LED, symbol Cherry_MX:Cherry-MX-RGB-0605
- added R1, R2, R3, R4, R5, R6: 150R, Resistor_SMD:R_0603_1608Metric, symbol Device:R
- added R50, R52, R53: 1k, Resistor_THT:R_Axial_DIN0204_L3.6mm_D1.6mm_P5.08mm_Horizontal, symbol Device:R_US
- added U1: 74HC595, Package_SO:SOIC-16W_5.3x10.2mm_P1.27mm, symbol 74xx:74HC595
Connections:
- net GND: now also R7.2, R8.2, C1.1, Eraser1.2, Play_Paper1.2, Play_Point1.2, Play_Pouch1.2, R1.2, R2.2, R3.2, R4.2, R5.2, R50.2, R52.2, R53.2, R6.2, Rec_Paper1.2, Rec_Point1.2, Rec_Pouch1.2, Smudger1.2, U1.13 (~{OE}), U1.8 (GND), U1.9 (QH')
- net LED_1: now also Eraser1.3 (A), U1.15 (QA); no longer R7.1
- net LED_2: now also Smudger1.3 (A), U1.1 (QB); no longer R8.1
- net LED_3: now also Rec_Pouch1.3 (A), U1.3 (QD)
- net LED_4: now also Play_Pouch1.3 (A), U1.2 (QC)
- net LED_5: now also Rec_Paper1.3 (A), U1.4 (QE)
- net LED_6: now also Play_Paper1.3 (A), U1.5 (QF)
- net LED_7: now also Rec_Point1.3 (A), U1.6 (QG)
- net LED_8: now also Play_Point1.3 (A), U1.7 (QH)
- new net: D2.1 (K), R50.1
- new net: R5.1, Smudger1.4 (C)
- new net: R6.1, Rec_Pouch1.4 (C)
- new net: Play_Paper1.4 (C), R4.1
- new net: D5.1 (K), R53.1
- new net: R1.1, Rec_Point1.4 (C)
- new net: Play_Point1.4 (C), R2.1
- new net: D4.1 (K), R52.1
- new net: Eraser1.4 (C), R8.1
- new net: R3.1, Rec_Paper1.4 (C)
- new net: Play_Pouch1.4 (C), R7.1
- new net 595_Data: U1.14 (SER)
- new net Button_Play_Palette: Play_Pouch1.1
- new net Button_Play_Paper: Play_Paper1.1
- new net Button_Play_Pattern: Smudger1.1
- new net Button_Play_Point: Play_Point1.1
- new net Button_Rec_Palette: Rec_Pouch1.1
- new net Button_Rec_Paper: Rec_Paper1.1
- new net Button_Rec_Pattern: Eraser1.1
- new net Button_Rec_Point: Rec_Point1.1
- new net CLK: U1.11 (SRCLK)
- new net LATCH: U1.12 (RCLK)
- new net Lid_On: D5.2 (A)
- new net VCC: C1.2, U1.10 (~{SRCLR}), U1.16 (VCC)
- new net c.o.t.l.: D4.2 (A)
- new net composition_LED: D2.2 (A)
Other:
- note removed: "Only buttons that can be latched need LEDS, this includes all mod buttons and discludes Empty and Settings. But since there are 16 leds for buttons plus 16 more for modes and side buttons, conservation of leds can be thrown out as a 3rd chip is then required. So no conservation of leds necessary"
- note removed: "was 140R for all LED resistors but not in stock"
